File: NeoMBB/Control.kicad_sch (KiCad schematic)
At the start: 20 parts, among them J29 Conn_01x02_Pin

Commit message: MBB Reverse engineering bs
Parts:
- removed C132: 100nF, Capacitor_SMD:C_1210_3225Metric_Pad1.33x2.70mm_HandSolder, symbol Device:C
- removed C133: 10uF, Capacitor_SMD:C_1210_3225Metric_Pad1.33x2.70mm_HandSolder, symbol Device:C
- removed J29: Conn_01x02_Pin, Connector_PinHeader_2.54mm:PinHeader_1x02_P2.54mm_Vertical, symbol Connector:Conn_01x02_Pin
- removed R12: 0, Resistor_SMD:R_1210_3225Metric_Pad1.30x2.65mm_HandSolder, symbol Device:R
- removed TP21, TP22, TP23, TP24, TP25, TP26, TP27, TP28, TP29, TP30, TP31, TP32, TP33, TP34, TP35: TestPoint, TestPoint:TestPoint_Loop_D2.54mm_Drill1.5mm_Beaded, symbol Connector:TestPoint
- added H1, H2, H3, H4: MountingHole, MountingHole:MountingHole_5.3mm_M5, symbol Mechanical:MountingHole
- added IC15, IC9: MCP23S17-E_SO, InverterCom:SOIC127P1030X265-28N, symbol InverterCom:MCP23S17-E_SO
- added J4: TBP01R2-508-04BE, InverterCom:SHDR4W100P0X508_1X4_2192X850X1200P, symbol InverterCom:TBP01R2-508-04BE
- added JP1, JP2, JP3, JP4: Jumper_2_Open, Jumper:SolderJumper-3_P2.0mm_Open_TrianglePad1.0x1.5mm, symbol Jumper:Jumper_2_Open
- A1: footprint InverterCom:RaspberryPi_Pico_Common_Unspecified -> Module:RaspberryPi_Pico_Common_THT
Connections:
- net GND_A is gone; now on net DIAG_GND: A1.13 (GND), A1.18 (GND), A1.23 (GND), A1.28 (GND), A1.3 (GND), A1.38 (GND), A1.8 (GND)
- net +3.3V_A: now also IC15.10 (VSS), IC15.9 (VDD), IC9.10 (VSS), IC9.9 (VDD)
- net MCP_SPI_RST2: now reaches A1.1 (GPIO0)
- net MCP_SPI_RST2: now also IC15.18 (~{RESET})
- net MCP_SPI_CS2: now reaches A1.2 (GPIO1)
- net MCP_SPI_CS2: now also IC15.11 (~{CS})
- net CAN4_INT: now reaches A1.22 (GPIO17)
- net MCP_SPI_CS: now reaches A1.24 (GPIO18)
- net MCP_SPI_CS: now also IC9.11 (~{CS})
- net MCP_SPI_INTA: now reaches A1.25 (GPIO19)
- net MCP_SPI_INTA: now also IC9.20 (INTA)
- net MCP_SPI_INTB: now reaches A1.26 (GPIO20)
- net MCP_SPI_INTB: now also IC9.19 (INTB)
- net MCP_SPI_RST: now reaches A1.27 (GPIO21)
- net MCP_SPI_RST: now also IC9.18 (~{RESET})
- net MTR_CTRL_ENABLE_SIGNAL: now reaches A1.29 (GPIO22)
- net DIAG_GND: now reaches A1.33 (AGND)
- net DIAG_GND: now also IC15.15 (A0), IC15.16 (A1), IC15.17 (A2), IC9.15 (A0), IC9.16 (A1), IC9.17 (A2), J4.1
- net GATE_DRIVER_FAULT_A renamed I_AMBIENT_TEMP_A
- net GATE_DRIVER_READY_A renamed UART_TX
- net GATE_DRIVER_RESET_A renamed UART_RX
- net RELAY1_A renamed CAN1_INT
- net RELAY2_A renamed CAN1_CS
- net RELAY3_A renamed CAN2_INT
- net SPI1_CAN_CS_A renamed MCP_SPI_INT2A
- net MCP_SPI_INT2A: now also IC15.20 (INTA)
- net SPI1_CAN_INT_A renamed MCP_SPI_INT2B
- net MCP_SPI_INT2B: now also IC15.19 (INTB)
- net SPI1_RX_A renamed CAN_SPI_RX
- net SPI1_SCK_A renamed CAN_SPI_SCK
- net SPI1_TX_A renamed CAN_SPI_TX
- net SPI2_CS_ADC1_A renamed CAN2_CS
- net SPI2_CS_ADC2_A renamed CAN3_INT
- net SPI2_CS_ADC3_A renamed CAN3_CS
- net SPI2_CS_ADC4_A renamed CAN4_CS
- net SPI2_RX_A renamed MCP_SPI_RX
- net MCP_SPI_RX: now also IC15.14 (SO), IC9.14 (SO)
- net SPI2_SCK_A renamed MCP_SPI_SCK
- net MCP_SPI_SCK: now also IC15.12 (SCK), IC9.12 (SCK)
- net SPI2_TX_A renamed MCP_SPI_TX
- net MCP_SPI_TX: now also IC15.13 (SI), IC9.13 (SI)
- new net +12V_A: J4.2
- new net CAN_2_H: J4.3
- new net CAN_2_L: J4.4
- new net I_ABS_INDICATOR_A: IC15.5 (GPB4)
- new net I_ABS_OFF_A: IC15.6 (GPB5)
- new net I_BRAKE_SWITCH_A: IC9.4 (GPB3)
- new net I_EXT_CHG_ENABLE0_A: IC15.28 (GPA7)
- new net I_EXT_CHG_ENABLE1_A: IC15.27 (GPA6)
- new net I_HVIL_STATUS_A: IC15.26 (GPA5)
- new net I_KEY_ON_A: IC9.3 (GPB2)
- new net I_KICKSTAND_SWITCH_A: IC9.2 (GPB1)
- new net I_MOTOR_START_SW_A: IC9.28 (GPA7)
- new net I_MOTOR_STOP_SW_A: IC9.1 (GPB0)
- new net I_OBC_ATTACHED_A: IC15.3 (GPB2)
- new net I_SYSTEM_ON_REF_A: IC9.27 (GPA6)
- new net I_THROTTLE_ENABLE_A: IC9.5 (GPB4)
- new net Isolated Canbus Module/CAN_JUMPER_A: JP1.2 (B)
- new net Isolated Canbus Module/CAN_JUMPER_B: JP1.1 (A)
- new net Isolated Canbus Module1/CAN_JUMPER_A: JP2.2 (B)
- new net Isolated Canbus Module1/CAN_JUMPER_B: JP2.1 (A)
- new net Isolated Canbus Module2/CAN_JUMPER_A: JP3.2 (B)
- new net Isolated Canbus Module2/CAN_JUMPER_B: JP3.1 (A)
- new net Isolated Canbus Module3/CAN_JUMPER_A: JP4.2 (B)
- new net Isolated Canbus Module3/CAN_JUMPER_B: JP4.1 (A)
- new net O_ABS_PWR_ENABLE_A: IC15.7 (GPB6)
- new net O_DASH_ABS_A: IC9.25 (GPA4)
- new net O_DASH_ARMED_A: IC9.24 (GPA3)
- new net O_DASH_CHG_A: IC9.23 (GPA2)
- new net O_DASH_CHG_RED_A: IC9.22 (GPA1)
- new net O_DASH_CHK_ENG_A: IC9.21 (GPA0)
- new net O_DASH_OVERTEMP_A: IC15.1 (GPB0)
- new net O_DASH_SYSWARN_A: IC15.2 (GPB1)
- new net O_DCDC_ENABLE_A: IC9.7 (GPB6)
- new net O_OBC_ENABLE_A: IC15.4 (GPB3)
- new net O_SEVCON_ENABLE_A: IC9.8 (GPB7)
- new net O_SEVCON_NEUTRAL_A: IC9.6 (GPB5)
- new net O_SYSTEM_ON_A: IC9.26 (GPA5)
- no-connect marks 5 -> 2
Other:
- added sheet Isolated Canbus Module (IsolatedCanbus.kicad_sch)
- added sheet Isolated Canbus Module1 (IsolatedCanbus.kicad_sch)
- added sheet Isolated Canbus Module2 (IsolatedCanbus.kicad_sch)
- added sheet Isolated Canbus Module3 (IsolatedCanbus.kicad_sch)
- note added: "12v chademo board connector"
- note added: "DIAG GND IS BONDED TO GND_A"
- note removed: "UART Debug Header"
