File: NeoMBB/IsolatedCanbus.kicad_sch (KiCad schematic)
At the start: 20 parts, among them IC1 MCP2515-e_ST, IC2 ISO1042BDWVR, Y1 8MHz

Commit message: MBB Reverse engineering bs
Parts:
- renumbered C1 to C44, C2 to C45, C3 to C46, C4 to C47, C5 to C48, C6 to C49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
