File: NeoMBB/MainBoard.kicad_sch (KiCad schematic)
At the start: 71 parts, among them IC9 MCP23S17-E_SO, J1 MX23A34NF1, J2 MX23A40NF1, J3 TBP01R1-508-08BE, J4 TBP01R2-508-04BE, J5 TBP01R2-508-04BE, Q1 SIHFR120-GE3, Q2 SIHFR120-GE3, U1 TCMT1100, U11 TCMT1100, U12 BTS462TATMA1, U2 TCMT1100, U3 TCMT1100, U4 TCMT1100, U5 BTS462TATMA1, U6 TCMT1100, U7 TCMT1100, U9 TCMT1100

Commit message: Probed Zero wiring harness
Parts:
- removed C27, C28, C29, C30, C31, C32, C33, C34, C35, C36, C37, C38, C39, C40, C41, C42: UCM1H101MCL1GS, CAPAE660X800N, symbol InverterCom:UCM1H101MCL1GS
- removed D1, D2, D3, D4: SM6T15A, Diode_SMD:D_SMB, symbol Diode:SM6T15A
- removed J3: TBP01R1-508-08BE, SHDR8W100P0X508_1X8_4224X1200X890P, symbol InverterCom:TBP01R1-508-08BE
- removed J5: TBP01R2-508-04BE, SHDR4W100P0X508_1X4_2192X850X1200P, symbol InverterCom:TBP01R2-508-04BE
- removed PS1: SCW20A-12, SCW20A12, symbol InverterCom:SCW20A-12
- removed PS4: R-78K3.3-1.0, R78K3310, symbol InverterCom:R-78K3.3-1.0
- removed Q1, Q2: SIHFR120-GE3, InverterCom:SIHFR120GE3, symbol InverterCom:SIHFR120-GE3
- removed R12, R16, R19, R24, R5, R7: 1k, Resistor_SMD:R_1210_3225Metric_Pad1.30x2.65mm_HandSolder, symbol Device:R
- removed R13, R14, R15, R17, R18, R20, R21, R25, R26, R6, R8: 4.7k, Resistor_SMD:R_1210_3225Metric_Pad1.30x2.65mm_HandSolder, symbol Device:R
- removed R22, R23: 120, Resistor_SMD:R_1210_3225Metric_Pad1.30x2.65mm_HandSolder, symbol Device:R
- removed U1, U11, U2, U3, U4, U6, U7, U9: TCMT1100, Package_SO:SOP-4_4.4x2.6mm_P1.27mm, symbol Isolator:TCMT1100
- removed U12, U5: BTS462TATMA1, Package_TO_SOT_SMD:TO-252-4, symbol Power_Management:BTS462TATMA1
- added J3: TBP02R2W-381-06BE, InverterCom:TBP02R2W38106BE, symbol InverterCom:TBP02R2W-381-06BE
- added PS1: OKI-78SR-5_1.5-W36E-C, InverterCom:OKI78SR515W36EC, symbol InverterCom:OKI-78SR-5_1.5-W36E-C
- added PS4: EC7BW-110S12, EC7BW110S12, symbol InverterCom:EC7BW-110S12
- added Q1: TBD62783AFG,EL, InverterCom:SOIC127P1030X245-18N, symbol InverterCom:TBD62783AFG,EL
- added R38: 10k, Resistor_SMD:R_1210_3225Metric_Pad1.30x2.65mm_HandSolder, symbol Device:R
- A1: footprint Module:RaspberryPi_Pico_Common_Unspecified -> Module:RaspberryPi_Pico_Common_THT
- IC9: footprint SOIC127P1030X265-28N -> InverterCom:SOIC127P1030X265-28N
- J1: footprint MX23A34NF1 -> InverterCom:MX23A34NF1
- J2: footprint MX23A40NF1 -> InverterCom:MX23A40NF1
- J4: footprint SHDR4W100P0X508_1X4_2192X850X1200P -> InverterCom:SHDR4W100P0X508_1X4_2192X850X1200P
- JP1, JP2, JP3, JP4: footprint (none) -> Jumper:SolderJumper-3_P2.0mm_Open_TrianglePad1.0x1.5mm
- R10: value 4.7k -> 0; now not fitted
- R11, R9: value 1k -> 0
Connections:
- net CHARGER_IN_DCP is gone; now on net HighSideOutputs/RELAY_3_COM: R10.2
- net DIAG_GND is gone; now on net 12V_GND: A1.13 (GND), A1.18 (GND), A1.23 (GND), A1.28 (GND), A1.3 (GND), A1.33 (AGND), A1.38 (GND), A1.8 (GND), IC9.15 (A0), IC9.16 (A1), IC9.17 (A2), J1.32, J2.31, J4.1, J4.3
- net HVIL_SOURCE is gone; now on net +5V_A: J2.14
- net KICKSTAND_SWITCH_SIG_5V is gone; now on net +5V_A: J1.27
- net KICKSTAND_SW_GND is gone; now on net 12V_GND: J1.12
- net MTR_CTRL_THROTTLE_5V_A is gone; now on net +5V_A: J2.34
- net MTR_CTRL_THROTTLE_5V_B is gone; now on net +5V_A: J2.37
- net +12V_A: now also R11.2, PS1.1 (+VIN), PS4.3 (+VOUT)
- net +3.3V_A: now also R38.1; no longer R10.1
- net 12V_GND: now also PS1.2 (GND), PS4.5 (-VOUT), Q1.10 (GND)
- net AMBIENT_TEMP: now also A1.31 (GPIO26_ADC0), R38.2
- net CAN2_+5V: now also J3.4
- net CAN2_GND: now also J3.3
- net CAN2_HIGH: now also J3.5
- net CAN2_LOW: now also J3.6
- net INST_CLUSTER_ABS: now also Q1.18 (O1)
- net INST_CLUSTER_CHARGING: now also Q1.16 (O3)
- net INST_CLUSTER_CHARG_RED: now also Q1.17 (O2)
- net INST_CLUSTER_CHK_ENG: now also Q1.12 (O7)
- net INST_CLUSTER_OVERTEMP: now also Q1.13 (O6)
- net INST_CLUSTER_SYS_ARMED: now also Q1.15 (O4)
- net INST_CLUSTER_SYS_WARN: now also Q1.14 (O5)
- net KEY_ON_12V: now also R11.1
- net MBB_LOW_PWR: now also R9.1, PS4.1 (+VIN)
- net POWER_PACK_GND: now also R10.1, PS4.2 (-VIN)
- net SIG_ABS_LIGHT: now reaches IC9.1 (GPB0)
- net SIG_ABS_LIGHT: now also Q1.1 (I1)
- net SIG_CHARGING_RED: now reaches IC9.2 (GPB1)
- net SIG_CHARGING_RED: now also Q1.2 (I2)
- net KICKSTAND_SW_FILTERED: now reaches IC9.21 (GPA0)
- net HVIL_SIG_FILTERED: now reaches IC9.22 (GPA1)
- net MTR_STOP_SW_SIGNAL: now reaches IC9.23 (GPA2)
- net START_SW_INPUT_SIGNAL: now reaches IC9.24 (GPA3)
- net BRAKE_SW_INPUT_SIGNAL: now reaches IC9.25 (GPA4)
- net ABS_ENABLE: now reaches IC9.26 (GPA5)
- net MTR_CTRL_NEUTRAL_SIGNAL: now reaches IC9.27 (GPA6)
- net DCDC_ENABLE_SIGNAL: now reaches IC9.28 (GPA7)
- net SIG_CHARGING: now reaches IC9.3 (GPB2)
- net SIG_CHARGING: now also Q1.3 (I3)
- net SIG_SYS_ARMED: now reaches IC9.4 (GPB3)
- net SIG_SYS_ARMED: now also Q1.4 (I4)
- net SIG_SYS_WARN: now reaches IC9.5 (GPB4)
- net SIG_SYS_WARN: now also Q1.5 (I5)
- net SIG_OVERTEMP: now reaches IC9.6 (GPB5)
- net SIG_OVERTEMP: now also Q1.6 (I6)
- net SIG_CHECK_ENG: now reaches IC9.7 (GPB6)
- net SIG_CHECK_ENG: now also Q1.7 (I7)
- net SYSTEM_ON_SIGNAL: now reaches IC9.8 (GPB7)
- net SYSTEM_ON_SIGNAL: now also Q1.8 (I8)
- net HighSideOutputs/RELAY_3_COM: now reaches R9.2
- net MTR_CTRL_ENABLE_SIGNAL: now reaches A1.29 (GPIO22)
- removed net +12V_CHAdeMO: R11.1, R9.1
- net EXT_SWITCH_5V renamed +5V_A
- net +5V_A: now also PS1.3 (+VOUT), Q1.9 (VCC)
- new net SYSTEM_ON_OUTPUT: Q1.11 (O8)
- no-connect marks 12 -> 25
Other:
- added sheet HighSideOutputs (HighSideOutputs.kicad_sch)
- added sheet VoltageSenseInputStage_Quad (VoltageSenseInputStage4.kicad_sch)
- added sheet VoltageSenseInputStage_Quad1 (VoltageSenseInputStage4.kicad_sch)
- note added: "<-- We can attach this to diginow instead of calex onboard crap, has side benefit of not cooking the battery unlike the stock calex"
- note added: "DRIVES THE +5V DISPLAY INDICATOR LAMPS THESE TAKE ~30mA EACH"
- note added: "We're just not gonna deal with this stuff"
- note removed: "------ CHARGER SIDE ------"
- note removed: "------ VEHICLE SIDE ------"
- note removed: "ALLOWS VEHICLE PULL DCP TO GND TO ENABLE"
- note removed: "CONTACTOR +12V CONNECTOR"
- note removed: "CONTACTOR DRIVER WE DO NOT DRIVE CONTACTORS DIRECTLY INSTEAD THEY ARE DONE VIA SOFTWARE AND THIS DRIVER"
- note removed: "DETECT IF CONNECTOR INSERTED (PP)"
- note removed: "IS THIS 12V? (REF'D TO INST_CLUSTER_GND) HOW MANY mA?"
- note removed: "MONITOR SS1 AND SS2 SS1 MONITORS FROM SS1 TO FG SS2 MONITORS FROM SS1 TO SS2"
- note removed: "MONITORS DCP ON CHARGER SIDE"
- note removed: "SS1 HIGH SIDE SWITCH (ALLOWS SS1 TO BE PULLED TO 12V)"
- note removed: "SS2 LOW SIDE SWITCH PULLS SS2 TO FG"
- note removed: "TERMINAL BLOCK TO CHADEMO SIGNAL CONNECTOR"
- note removed: "WHAT VOLTAGES DO THESE TAKE? ARE THEY IN/OUT?"
- note removed: "~200 OHM RESISTOR FOR PROXIMITY PIN, ONLY SOLDER THIS ON CHARGER SIDE THE EXACT VALUE IS NOT IMPORTANT, REUSING 2X 120 OHMS TO SAVE PARTS"
- moved on the sheet: J1, J2

Commit message: MBB Reverse engineering bs
Parts:
- removed A1: RaspberryPi_Pico, Module:RaspberryPi_Pico_Common_THT, symbol MCU_Module:RaspberryPi_Pico
- removed H1, H2, H3, H4: MountingHole, MountingHole:MountingHole_5.3mm_M5, symbol Mechanical:MountingHole
- removed IC9: MCP23S17-E_SO, InverterCom:SOIC127P1030X265-28N, symbol InverterCom:MCP23S17-E_SO
- removed J3: TBP02R2W-381-06BE, InverterCom:TBP02R2W38106BE, symbol InverterCom:TBP02R2W-381-06BE
- removed J4: TBP01R2-508-04BE, InverterCom:SHDR4W100P0X508_1X4_2192X850X1200P, symbol InverterCom:TBP01R2-508-04BE
- removed JP1, JP2, JP3, JP4: Jumper_2_Open, Jumper:SolderJumper-3_P2.0mm_Open_TrianglePad1.0x1.5mm, symbol Jumper:Jumper_2_Open
- removed PS1: OKI-78SR-5_1.5-W36E-C, InverterCom:OKI78SR515W36EC, symbol InverterCom:OKI-78SR-5_1.5-W36E-C
- removed PS4: EC7BW-110S12, EC7BW110S12, symbol InverterCom:EC7BW-110S12
- removed Q1: TBD62783AFG,EL, InverterCom:SOIC127P1030X245-18N, symbol InverterCom:TBD62783AFG,EL
- removed R10, R11, R9: 0, Resistor_SMD:R_1210_3225Metric_Pad1.30x2.65mm_HandSolder, symbol Device:R
- removed R38: 10k, Resistor_SMD:R_1210_3225Metric_Pad1.30x2.65mm_HandSolder, symbol Device:R
- added R53: 0, Resistor_SMD:R_1210_3225Metric_Pad1.30x2.65mm_HandSolder, symbol Device:R
Connections:
- net +5V_A: no longer J1.23, J1.27, J2.14, J2.34, J2.37
- net IO_SYSTEM_ON_REF_+5V_C: now reaches J1.8
- removed net 12V_GND: J1.12, J1.29, J1.32, J2.31
- net ABS_HCU_VOLTAGE renamed OUTPUT_ABS_HCU_+12V_A
- net ABS_INDICATOR_INPUT renamed INPUT_ABS_INDICATOR_+12V_A
- net ABS_OFF renamed INPUT_ABS_OFF_+12V_A
- net AMBIENT_TEMP renamed INPUT_AMBIENT_TEMP_A
- net BATTERY_THROTTLE_ENABLE renamed INPUT_BATTERY_THROTTLE_ENABLE_+5V_A
- net BRAKE_SW_INPUT renamed INPUT_BRAKE_SWITCH_+12V_A
- net CAN0_+5V renamed OUTPUT_CAN0_+5V_E
- net CAN0_GND renamed CAN0_GND_E
- net CAN0_HIGH renamed IO_CAN0_HIGH_E
- net CAN0_LOW renamed IO_CAN0_LOW_E
- net CAN1_GND renamed CAN1_GND_F
- net CAN1_HIGH renamed IO_CAN1_HIGH_F
- net CAN1_LOW renamed IO_CAN1_LOW_F
- net CAN2_+5V renamed CAN2_+5V_G
- net CAN2_GND renamed CAN2_GND_G
- net CAN2_HIGH renamed IO_CAN2_HIGH_G
- net CAN2_LOW renamed IO_CAN2_LOW_G
- net DC/DC_CONV_ENABLE renamed OUTPUT_DCDC_ENABLE_+VBATT_C
- net EXT_CHARGER_ENABLE_0 renamed INPUT_EXT_CHARGER_ENABLE_0_+VBATT_C
- net EXT_CHARGER_ENABLE_1 renamed INPUT_EXT_CHARGER_ENABLE_1_+VBATT_C
- net EXT_SW_5V renamed OUTPUT_START_SWITCH_+5V_D
- net FUEL_GATE_5V_REF renamed OUTPUT_INST_CLUST_SUPPLY_+5V_B
- net FUSE1_ABS4KEY_12VPOS renamed INPUT_ABS_HCU_POWER_+12V_A
- net HVIL_RETURN renamed INPUT_HVIL_RETURN_+5V_A
- net INST_CLUSTER_ABS renamed OUTPUT_INST_CLUST_ABS_+5V_B
- net INST_CLUSTER_CHARGING renamed OUTPUT_INST_CLUST_CHG_+5V_B
- net INST_CLUSTER_CHARG_RED renamed OUTPUT_INST_CLUST_CHG_RED_+5V_B
- net INST_CLUSTER_CHK_ENG renamed OUTPUT_INST_CLUST_CHK_ENG_+5V_B
- net INST_CLUSTER_OVERTEMP renamed OUTPUT_INST_CLUST_OVERTEMP_+5V_B
- net INST_CLUSTER_SYS_ARMED renamed OUTPUT_INST_CLUST_ARMED_+5V_B
- net INST_CLUSTER_SYS_WARN renamed OUTPUT_INST_CLUST_SYS_WARN_+5V_B
- net KEY_ON_12V renamed KEY_ON_+12V_A
- net KICKSTAND_SW_SIG renamed INPUT_KICKSTAND_SWITCH_+5V_D
- net MBB_LOW_PWR renamed TRBATT_B+_C
- net MOTOR_CONTR_+24V_IN renamed NC_INPUT_SEVCON_+24V_C
- net MOTOR_CONTR_CAN_HIGH renamed IO_MOTOR_CONTR_CAN_HIGH_C
- net MOTOR_CONTR_CAN_LOW renamed IO_MOTOR_CONTR_CAN_LOW_C
- net MOTOR_CONTR_GND renamed SEVCON_GND_C
- net MTR_CTRL_ENABLE renamed OUTPUT_SEVCON_ENABLE_+VBATT_C
- net MTR_CTRL_NEUTRAL renamed OUTPUT_SEVCON_NEUTRAL_+VBATT_C
- net MTR_STOP_SW_IN renamed INPUT_MTR_STOP_SWITCH_SIGNAL_+5V_D
- net POWER_PACK_GND renamed TRBATT_GND_C
- net START_SW_INPUT renamed INPUT_START_SWITCH_SENSE_+5V_D
- net SYSTEM_ON_INPUT renamed OUTPUT_SYSTEM_ON_+5V_C
- new net +12V_GND_A: J1.29, R53.2
- new net DIAG_GND: J2.31
- new net GND_A: R53.1
- new net INST_CLUSTER_GND_B: J1.32
- new net KICKSTAND_SWITCH_GND_D: J1.12
- new net OUTPUT_HVIL_SOURCE_+5V_A: J2.14
- new net OUTPUT_KICKSTAND_SWITCH_+5V_D: J1.27
- new net OUTPUT_MTR_CTRL_THROTTLE1_+5V_C: J2.34
- new net OUTPUT_MTR_CTRL_THROTTLE2_+5V_C: J2.37
- new net OUTPUT_MTR_STOP_SWITCH_+5V_D: J1.23
- no-connect marks 25 -> 16
Other:
- removed sheet HighSideOutputs
- removed sheet Isolated Canbus Module
- removed sheet Isolated Canbus Module1
- removed sheet Isolated Canbus Module2
- removed sheet Isolated Canbus Module3
- removed sheet VoltageSenseInputStage_Quad
- removed sheet VoltageSenseInputStage_Quad1
- added sheet ABS Interface (ABS.kicad_sch)
- added sheet Charger Interface (ChargerInterface.kicad_sch)
- added sheet Control (Control.kicad_sch)
- added sheet Dash Interface (DashInterface.kicad_sch)
- added sheet High Voltage Interlock (HVIL.kicad_sch)
- added sheet Inverter Interface (InverterInterface.kicad_sch)
- added sheet Power (Power.kicad_sch)
- added sheet Sensor IO (SensorIO.kicad_sch)
- note removed: "12v input connector"
- note removed: "<-- We can attach this to diginow instead of calex onboard crap, has side benefit of not cooking the battery unlike the stock calex"
- note removed: "DRIVES THE +5V DISPLAY INDICATOR LAMPS THESE TAKE ~30mA EACH"
- note removed: "THESE TOO, HOW ARE THESE DRIVEN? ARE THEY HIGH SIDE SWITCH, LOW SIDE? INPUT? OUTPUT? WHAT CURRENT, ETC?"
- note removed: "We're just not gonna deal with this stuff"
- moved on the sheet: J1, J2
